File: C64NIKI2.kicad_sch (KiCad schematic)
At the start: 25 parts, among them J1 C64-EXP, Q1 BC237, SW1 FREEZE, SW2 RESET, U1 74LS74, U2 74LS163, U3 74LS125, U4 74LS05, U5 74LS174, U6 27C256

Commit message: work in progress
Parts:
- Q1: footprint Package_TO_SOT_THT:TO-92_Inline -> Package_TO_SOT_THT:TO-92_Wide
Changed lines of the file:
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@@
       (effects (font (size 1.27 1.27)) (justify left))
     )
-    (property "Footprint" "Package_TO_SOT_THT:TO-92_Inline" (at 121.92 80.645 0)
+    (property "Footprint" "Package_TO_SOT_THT:TO-92_Wide" (at 121.92 80.645 0)
       (effects (font (size 1.27 1.27) italic) (justify left) hide)
     )

Commit message: first release
Parts:
- added JP1, JP2: 1-2 = 27C - 2-3 = 28C, C64NIKI2:BottomSolderJumper-3_P1.3mm_Bridged2Bar12_Pad1.0x1.5mm_NumberLabels, symbol Jumper:Jumper_3_Bridged12
Connections:
- net GND: now also U4.11, U4.13, U4.5, U4.9
- net VCC: now also JP1.1 (A), JP2.3 (B); no longer U6.1 (VPP)
- net at U5.2 (Q0): now also JP1.3 (B), JP2.1 (A); no longer U6.27 (A14)
- net EXP_10 renamed IO2
- net EXP_11 renamed ROML
- net EXP_4 renamed IRQ
- net EXP_5 renamed RW
- net EXP_7 renamed IO1
- net EXP_8 renamed GAME
- net EXP_9 renamed EXROM
- net EXP_B renamed ROMH
- net EXP_C renamed RESET
- net EXP_D renamed NMI
- net EXP_E renamed PHI2
- new net: JP2.2 (C), U6.27 (A14)
- new net: JP1.2 (C), U6.1 (VPP)
- no-connect marks 20 -> 16
Other:
- title: (none) -> C64 NIKI2
- moved on the sheet: U4D, U4F
